Commit message: a

File: examples/car_dae.urdf (robot description, URDF)
Before this commit: robot car_model, 5 links, 4 joints
Links:
- added link steer_fl_link, mass 0.5
- added link steer_fr_link, mass 0.5
- added link susp_fl, mass 1.0
- added link susp_fr, mass 1.0
- added link susp_rl, mass 1.0
- added link susp_rr, mass 1.0
- link car_body: mass 8.0 -> 1200.0; geometry collision box size=2.5 1.2 0.5; visual box size=2.5 1.2 0.5
- link wheel_fl: mass 1.5 -> 20.0; geometry collision cylinder length=0.2 radius=0.35; visual cylinder length=0.2 radius=0.35
- link wheel_fr: mass 1.5 -> 20.0; geometry collision cylinder length=0.2 radius=0.35; visual cylinder length=0.2 radius=0.35
- link wheel_rl: mass 1.5 -> 20.0; geometry collision cylinder length=0.2 radius=0.35; visual cylinder length=0.2 radius=0.35
- link wheel_rr: mass 1.5 -> 20.0; geometry collision cylinder length=0.2 radius=0.35; visual cylinder length=0.2 radius=0.35
Joints:
- removed joint joint_fl
- removed joint joint_fr
- removed joint joint_rl
- removed joint joint_rr
- added joint rear_rl: type continuous, parent susp_rl, child wheel_rl, origin xyz=0 0 -0.35 rpy=0 0 0, axis 0 1 0
- added joint rear_rr: type continuous, parent susp_rr, child wheel_rr, origin xyz=0 0 -0.35 rpy=0 0 0, axis 0 1 0
- added joint steer_fl: type revolute, parent susp_fl, child steer_fl_link, origin xyz=0 0 -0.35 rpy=0 0 0, axis 0 0 1, limit lower=-0.6 upper=0.6 effort=500 velocity=2
- added joint steer_fr: type revolute, parent susp_fr, child steer_fr_link, origin xyz=0 0 -0.35 rpy=0 0 0, axis 0 0 1, limit lower=-0.6 upper=0.6 effort=500 velocity=2
- added joint susp_fl_joint: type fixed, parent car_body, child susp_fl, origin xyz=1.2 -0.6 -0.25 rpy=0 0 0
- added joint susp_fr_joint: type fixed, parent car_body, child susp_fr, origin xyz=1.2 0.6 -0.25 rpy=0 0 0
- added joint susp_rl_joint: type fixed, parent car_body, child susp_rl, origin xyz=-1.2 -0.6 -0.25 rpy=0 0 0
- added joint susp_rr_joint: type fixed, parent car_body, child susp_rr, origin xyz=-1.2 0.6 -0.25 rpy=0 0 0
- added joint wheel_fl_rotate: type continuous, parent steer_fl_link, child wheel_fl, origin xyz=0 0 0 rpy=0 0 0, axis 0 1 0
- added joint wheel_fr_rotate: type continuous, parent steer_fr_link, child wheel_fr, origin xyz=0 0 0 rpy=0 0 0, axis 0 1 0
